Commit message: fix dimensions

File: gobilda_ws/src/gobilda_robot/description/urdf/gobilda_description.urdf.xacro (robot description, xacro)
@@ -5,10 +5,10 @@
   <xacro:property name="PI" value="3.1415926535897931"/>
   <xacro:property name="base_mass" value="0.3" /> <!-- arbitrary value for base mass -->
-  <xacro:property name="base_width" value="0.1" />
-  <xacro:property name="base_length" value="0.1" />
-  <xacro:property name="base_height" value="0.05" />
+  <xacro:property name="base_width" value="0.467" />
+  <xacro:property name="base_length" value="0.433" />
+  <xacro:property name="base_height" value="0.095" />
   <xacro:property name="wheel_mass" value="0.3" /> <!-- arbitrary value for wheel mass -->
-  <xacro:property name="wheel_len" value="0.020" />
-  <xacro:property name="wheel_radius" value="0.015" />
+  <xacro:property name="wheel_len" value="0.24" />
+  <xacro:property name="wheel_radius" value="0.0475" />
   <xacro:property name="z_offset" value="-${base_height/2}" /> <!-- Space btw top of beam and the each joint -->
   <!-- Base Link -->
